Commit message: added convex hulls

File: urdf/bit_xuanyuan.urdf (robot description, URDF)
Before this commit: robot bit_xuanyuan, 43 links, 42 joints
Links:
- removed link L_ankle_6 axis
- removed link L_wrist_6 axis
- removed link R_ankle_6 axis
- removed link R_wrist_6 axis
- added link L_ankle_6_axis, mass 0.507659863952687; collision mesh filename=package://bit_xuanyuan_description/meshes/L_ankle_6_axis.STL; visual mesh filename=package://bit_xuanyuan_description/meshes/L_ankle_6_axis.STL
- added link L_wrist_6_axis, mass 0.236120679342982; collision mesh filename=package://bit_xuanyuan_description/meshes/L_wrist_6_axis.STL; visual mesh filename=package://bit_xuanyuan_description/meshes/L_wrist_6_axis.STL
- added link R_ankle_6_axis, mass 0.507659863952688; collision mesh filename=package://bit_xuanyuan_description/meshes/R_ankle_6_axis.STL; visual mesh filename=package://bit_xuanyuan_description/meshes/R_ankle_6_axis.STL
- added link R_wrist_6_axis, mass 0.236120679342982; collision mesh filename=package://bit_xuanyuan_description/meshes/R_wrist_6_axis.STL; visual mesh filename=package://bit_xuanyuan_description/meshes/R_wrist_6_axis.STL
Joints:
- removed joint L_ankle_6 axis
- removed joint L_wrist_6 axis
- removed joint R_ankle_6 axis
- removed joint R_wrist_6 axis
- added joint L_ankle_6_axis: type fixed, parent L_ankle_2, child L_ankle_6_axis, origin xyz=0 0.115721608105073 0.0590748593972637 rpy=-1.5707963267949 0 -3.14159265358979, axis 0 0 0
- added joint L_wrist_6_axis: type fixed, parent L_wrist_2, child L_wrist_6_axis, origin xyz=0 -0.045 -0.025 rpy=1.5708 0 3.1416, axis 0 0 0
- added joint R_ankle_6_axis: type fixed, parent R_ankle_2, child R_ankle_6_axis, origin xyz=0 0.101737731329006 0.0590748593972759 rpy=-1.5707963267949 0 3.14159265358979, axis 0 0 0
- added joint R_wrist_6_axis: type fixed, parent R_wrist_2, child R_wrist_6_axis, origin xyz=0 -0.0545 0.024999999999999 rpy=-1.5707963267949 0 0, axis 0 0 0
- joint L_foot: parent L_ankle_6 axis -> L_ankle_6_axis
- joint L_hand: parent L_wrist_6 axis -> L_wrist_6_axis
- joint R_foot: parent R_ankle_6 axis -> R_ankle_6_axis
- joint R_hand: parent R_wrist_6 axis -> R_wrist_6_axis

Commit message: added a torso link and made it face +x direction instead of -y

File: urdf/bit_xuanyuan.urdf (robot description, URDF)
Before this commit: robot bit_xuanyuan, 43 links, 42 joints
Links:
- added link torso, mass 26.3712421112853; collision mesh filename=package://bit_xuanyuan_description/meshes/torso.STL; visual mesh filename=package://bit_xuanyuan_description/meshes/torso.STL
- link base_link: mass 26.3712421112853 -> None; geometry 
Joints:
- added joint waist: type fixed, parent base_link, child torso, origin xyz=0 0 0 rpy=0 0 0
- joint L_shoulder_1: origin xyz=0.248151606851778 -0.0263301173710569 0.208999973477994 rpy=1.5707963267949 0 1.5707963267949 -> xyz=0.0263301173710569 0.248151606851778 0.208999973477994 rpy=1.5707963267949 0 3.14159265; parent base_link -> torso
- joint R_shoulder_1: origin xyz=-0.248151606851778 -0.0263301173710569 0.209000026522007 rpy=1.5707963267949 0 -1.5707963267949 -> xyz=0.0263301173710569 -0.248151606851778 0.209000026522007 rpy=1.5707963267949 0 0; parent base_link -> torso
- joint waist_0: origin xyz=0.0751588565074892 0 -0.0749999999999999 rpy=1.5707963267949 0 1.5707963267949 -> xyz=0 0.0751588565074892 -0.0749999999999999 rpy=1.5707963267949 0 3.14159265; parent base_link -> torso

Commit message: Fix (some) joint axis

File: urdf/bit_xuanyuan.urdf (robot description, URDF)
Before this commit: robot bit_xuanyuan, 44 links, 43 joints
Joints:
- joint L_elbow_1: axis 0 0 1 -> 0 0 -1
- joint L_knee_1: axis 0 0 1 -> 0 0 -1
- joint R_elbow_1: axis 0 0 1 -> 0 0 -1

Commit message: Fix limits on R_elbow_1

File: urdf/bit_xuanyuan.urdf (robot description, URDF)
Before this commit: robot bit_xuanyuan, 44 links, 43 joints
Joints:
- joint R_elbow_1: limit lower=0 upper=2.255 effort=50 velocity=3.14 -> lower=-0.75 upper=2.255 effort=50 velocity=3.14

Commit message: Fix limits on L_ankle_1

File: urdf/bit_xuanyuan.urdf (robot description, URDF)
Before this commit: robot bit_xuanyuan, 44 links, 43 joints
Joints:
- joint L_ankle_1: limit lower=-0.4014 upper=1.5707 effort=70 velocity=1.57 -> lower=-1.5707 upper=0.4014 effort=70 velocity=1.57

Commit message: Fix mimic multiplier for gripper joints

File: urdf/bit_xuanyuan.urdf (robot description, URDF)
Before this commit: robot bit_xuanyuan, 44 links, 43 joints
Joints:
- joint L_gripper_2: mimic joint=L_gripper_1 multiplier=1 offset=0 -> joint=L_gripper_1 multiplier=-1 offset=0
- joint R_gripper_2: mimic joint=R_gripper_1 multiplier=1 offset=0 -> joint=R_gripper_1 multiplier=-1 offset=0

Commit message: changed waist_1's +x to be pointing forward

File: urdf/bit_xuanyuan.urdf (robot description, URDF)
Before this commit: robot bit_xuanyuan, 44 links, 43 joints
Joints:
- joint L_hip_1: origin xyz=-0.0874524045087781 0 0.0804896286305103 rpy=0 0 0 -> xyz=0 -0.0874524045087781 0.0804896286305103 rpy=0 0 1.5707963267949
- joint R_hip_1: origin xyz=0.0873497468913164 5.9130214832445E-05 0.0804842516395254 rpy=0 0 0 -> xyz=5.9130214832445E-05 0.0873497468913164 0.0804842516395254 rpy=0 0 1.5707963267949
- joint waist_1: origin xyz=0 -0.0460046428794829 -0.0751888646756264 rpy=1.5707963267949 1.5707963267949 0 -> xyz=0 -0.0460046428794829 -0.0751888646756264 rpy=1.5707963267949 3.1415926535 0

Commit message: magnify velocity limit

File: urdf/bit_xuanyuan.urdf (robot description, URDF)
Before this commit: robot bit_xuanyuan, 44 links, 43 joints
Joints:
- joint L_ankle_1: limit lower=-1.5707 upper=0.4014 effort=70 velocity=1.57 -> lower=-1.5707 upper=0.4014 effort=70 velocity=3.1415
- joint L_ankle_2: limit lower=-0.4886 upper=0.4886 effort=70 velocity=1.57 -> lower=-0.4886 upper=0.4886 effort=70 velocity=3.1415
- joint L_hip_1: limit lower=-3.14 upper=3.14 effort=300 velocity=1.57 -> lower=-3.14 upper=3.14 effort=300 velocity=3.1415
- joint L_hip_3: limit lower=-1.57 upper=1.57 effort=200 velocity=1.57 -> lower=-1.57 upper=1.57 effort=200 velocity=3.1415
- joint L_knee_1: limit lower=-2.7925 upper=0.1919 effort=150 velocity=1.57 -> lower=-2.7925 upper=0.1919 effort=150 velocity=3.1415
- joint L_knee_2: limit lower=-1.57 upper=1.57 effort=200 velocity=1.57 -> lower=-1.57 upper=1.57 effort=200 velocity=3.1415
- joint R_ankle_1: limit lower=-0.4014 upper=1.5707 effort=70 velocity=1.57 -> lower=-0.4014 upper=1.5707 effort=70 velocity=3.1415
- joint R_ankle_2: limit lower=-0.4886 upper=0.4886 effort=70 velocity=1.57 -> lower=-0.4886 upper=0.4886 effort=70 velocity=3.1415
- joint R_hip_1: limit lower=-3.14 upper=3.14 effort=300 velocity=1.57 -> lower=-3.14 upper=3.14 effort=300 velocity=3.1415
- joint R_hip_2: limit lower=-0.4188 upper=0.4188 effort=300 velocity=1.57 -> lower=-0.4188 upper=0.4188 effort=300 velocity=3.1415
- joint R_hip_3: limit lower=-1.57 upper=1.57 effort=300 velocity=1.57 -> lower=-1.57 upper=1.57 effort=300 velocity=3.1415
- joint R_knee_1: limit lower=-2.7925 upper=0.1919 effort=150 velocity=1.57 -> lower=-2.7925 upper=0.1919 effort=150 velocity=3.1415
- joint R_knee_2: limit lower=-1.57 upper=1.57 effort=200 velocity=1.57 -> lower=-1.57 upper=1.57 effort=200 velocity=3.1415
- joint waist_0: limit lower=-0.872 upper=0.872 effort=300 velocity=1.57 -> lower=-0.872 upper=0.872 effort=300 velocity=3.1415
- joint waist_1: limit lower=-0.872 upper=0.872 effort=300 velocity=1.57 -> lower=-0.872 upper=0.872 effort=300 velocity=3.1415

Commit message: Add LeftGripper and RightGripper
- Adjust velocity limits

File: urdf/bit_xuanyuan.urdf (robot description, URDF)
Before this commit: robot bit_xuanyuan, 44 links, 43 joints
Joints:
- joint L_gripper_1: limit lower=-0.01 upper=0.01 effort=200 velocity=1 -> lower=-0.01 upper=0.01 effort=200 velocity=0.015
- joint L_gripper_2: limit lower=-0.01 upper=0.01 effort=200 velocity=1 -> lower=-0.01 upper=0.01 effort=200 velocity=0.015
- joint R_gripper_1: limit lower=-0.01 upper=0.01 effort=200 velocity=1 -> lower=-0.01 upper=0.01 effort=200 velocity=0.015
- joint R_gripper_2: limit lower=-0.01 upper=0.01 effort=200 velocity=1 -> lower=-0.01 upper=0.01 effort=200 velocity=0.015

Commit message: Change gripper orientation to match real robot

File: urdf/bit_xuanyuan.urdf (robot description, URDF)
Before this commit: robot bit_xuanyuan, 44 links, 43 joints
Joints:
- joint L_hand: origin xyz=0 0 -0.0150000000000001 rpy=0 0 3.14159265358979 -> xyz=0.05 0 -0.04 rpy=-3.14 -1.57 0.0
- joint R_hand: origin xyz=0 0 -0.00550000000000006 rpy=0 0 3.14159265358979 -> xyz=-0.05 0 -0.03 rpy=-3.14 1.57 0.0

Commit message: updated joint max speed and effort according to the real robot config

File: urdf/bit_xuanyuan.urdf (robot description, URDF)
Before this commit: robot bit_xuanyuan, 44 links, 43 joints
Joints:
- joint L_ankle_1: limit lower=-1.5707 upper=0.4014 effort=70 velocity=3.1415 -> lower=-1.5707 upper=0.4014 effort=116 velocity=4.3
- joint L_ankle_2: limit lower=-0.4886 upper=0.4886 effort=70 velocity=3.1415 -> lower=-0.4886 upper=0.4886 effort=70 velocity=4.9
- joint L_elbow_1: limit lower=-0.75 upper=2.255 effort=50 velocity=3.14 -> lower=0 upper=1.745 effort=200 velocity=2.14
- joint L_elbow_2: limit lower=-1.5075 upper=4.7728 effort=50 velocity=3.14 -> lower=-1.5075 upper=4.7728 effort=20 velocity=10.14
- joint L_hip_1: limit lower=-3.14 upper=3.14 effort=300 velocity=3.1415 -> lower=-3.14 upper=3.14 effort=150 velocity=2.3
- joint L_hip_2: limit lower=-0.4188 upper=0.4188 effort=100 velocity=3.14 -> lower=-0.4188 upper=0.4188 effort=300 velocity=2.3
- joint L_hip_3: limit lower=-1.57 upper=1.57 effort=200 velocity=3.1415 -> lower=-1.57 upper=1.57 effort=179 velocity=3.0
- joint L_knee_1: limit lower=-2.7925 upper=0.1919 effort=150 velocity=3.1415 -> lower=-2.7925 upper=0.1919 effort=300 velocity=2.0
- joint L_knee_2: limit lower=-1.57 upper=1.57 effort=200 velocity=3.1415 -> lower=-1.57 upper=1.57 effort=65 velocity=7.0
- joint L_shoulder_1: limit lower=-3.14 upper=3.14 effort=100 velocity=3.14 -> lower=-2.62 upper=0.7 effort=150 velocity=3.14
- joint L_shoulder_2: limit lower=-0.91 upper=1.69 effort=100 velocity=3.14 -> lower=-1.31 upper=0.785 effort=200 velocity=1.57
- joint L_shoulder_3: limit lower=-1.57 upper=4.71 effort=75 velocity=3.14 -> lower=-1.483 upper=1.483 effort=100 velocity=5.97
- joint L_wrist_1: limit lower=-1.2 upper=1.2 effort=50 velocity=3.14 -> lower=-0.663 upper=0.663 effort=30 velocity=3.14
- joint L_wrist_2: limit lower=-0.75 upper=0.85 effort=50 velocity=3.14 -> lower=-0.75 upper=0.75 effort=50 velocity=3.14
- joint R_ankle_1: limit lower=-0.4014 upper=1.5707 effort=70 velocity=3.1415 -> lower=-0.4014 upper=1.5707 effort=116 velocity=4.3
- joint R_ankle_2: limit lower=-0.4886 upper=0.4886 effort=70 velocity=3.1415 -> lower=-0.4886 upper=0.4886 effort=70 velocity=4.9
- joint R_elbow_1: limit lower=-0.75 upper=2.255 effort=50 velocity=3.14 -> lower=0 upper=1.745 effort=200 velocity=2.14
- joint R_elbow_2: limit lower=-1.5072 upper=4.7728 effort=50 velocity=3.14 -> lower=-1.4835 upper=1.4835 effort=20 velocity=10.14
- joint R_hip_1: limit lower=-3.14 upper=3.14 effort=300 velocity=3.1415 -> lower=-3.14 upper=3.14 effort=150 velocity=2.3
- joint R_hip_2: limit lower=-0.4188 upper=0.4188 effort=300 velocity=3.1415 -> lower=-0.4188 upper=0.4188 effort=300 velocity=2.3
- joint R_hip_3: limit lower=-1.57 upper=1.57 effort=300 velocity=3.1415 -> lower=-1.57 upper=1.57 effort=179 velocity=3.0
- joint R_knee_1: limit lower=-2.7925 upper=0.1919 effort=150 velocity=3.1415 -> lower=-2.7925 upper=0.1919 effort=300 velocity=2.0
- joint R_knee_2: limit lower=-1.57 upper=1.57 effort=200 velocity=3.1415 -> lower=-1.57 upper=1.57 effort=60 velocity=7.1
- joint R_shoulder_1: limit lower=-3.14 upper=3.14 effort=150 velocity=3.14 -> lower=-1.047 upper=2.44346 effort=150 velocity=3.14
- joint R_shoulder_2: limit lower=-0.91 upper=1.69 effort=100 velocity=3.14 -> lower=-0.7854 upper=1.082 effort=200 velocity=1.57
- joint R_shoulder_3: limit lower=-4.71 upper=1.57 effort=75 velocity=3.14 -> lower=-1.535 upper=1.535 effort=75 velocity=5.97
- joint R_wrist_1: limit lower=-1.2 upper=1.2 effort=50 velocity=3.14 -> lower=-0.663 upper=0.663 effort=30 velocity=3.42
- joint R_wrist_2: limit lower=-0.75 upper=0.85 effort=50 velocity=3.14 -> lower=-0.75 upper=0.75 effort=30 velocity=3.42
- joint waist_0: limit lower=-0.872 upper=0.872 effort=300 velocity=3.1415 -> lower=-0.872 upper=0.872 effort=300 velocity=2.8
- joint waist_1: limit lower=-0.872 upper=0.872 effort=300 velocity=3.1415 -> lower=-0.872 upper=0.872 effort=220 velocity=2.5

Commit message: limitting waist pitch to 40 degrees (previous matx value is 50)

File: urdf/bit_xuanyuan.urdf (robot description, URDF)
Before this commit: robot bit_xuanyuan, 44 links, 43 joints
Joints:
- joint waist_0: limit lower=-0.872 upper=0.872 effort=300 velocity=2.8 -> lower=-0.7 upper=0.1 effort=300 velocity=2.8

Commit message: updated joint limits for upper body

File: urdf/bit_xuanyuan.urdf (robot description, URDF)
Before this commit: robot bit_xuanyuan, 44 links, 43 joints
Joints:
- joint L_ankle_1: limit lower=-0.436 upper=0.436 effort=116 velocity=4.3 -> lower=-0.4014 upper=0.4014 effort=116 velocity=4.3
- joint L_ankle_2: limit lower=-0.35 upper=0.35 effort=70 velocity=4.9 -> lower=-0.4014 upper=0.4014 effort=70 velocity=4.9
- joint R_ankle_1: limit lower=-0.436 upper=0.436 effort=116 velocity=4.3 -> lower=-0.4014 upper=0.4014 effort=116 velocity=4.3
- joint R_ankle_2: limit lower=-0.35 upper=0.35 effort=70 velocity=4.9 -> lower=-0.4014 upper=0.4014 effort=70 velocity=4.9

Commit message: updating joint limits;

File: urdf/bit_xuanyuan.urdf (robot description, URDF)
Before this commit: robot bit_xuanyuan, 44 links, 43 joints
Joints:
- joint L_ankle_1: limit lower=-1.5707 upper=0.4014 effort=116 velocity=4.3 -> lower=-0.4014 upper=0.4014 effort=116 velocity=4.3
- joint L_ankle_2: limit lower=-0.4886 upper=0.4886 effort=70 velocity=4.9 -> lower=-0.4014 upper=0.4014 effort=70 velocity=4.9
- joint L_hip_3: limit lower=-1.57 upper=1.57 effort=179 velocity=3.0 -> lower=-1.57 upper=0.6 effort=179 velocity=3.0
- joint L_wrist_1: limit lower=-0.663 upper=0.663 effort=30 velocity=3.14 -> lower=-0.63 upper=0.63 effort=30 velocity=3.14
- joint L_wrist_2: limit lower=-0.75 upper=0.75 effort=50 velocity=3.14 -> lower=-0.73 upper=0.73 effort=50 velocity=3.14
- joint R_ankle_1: limit lower=-0.4014 upper=1.5707 effort=116 velocity=4.3 -> lower=-0.4014 upper=0.4014 effort=116 velocity=4.3
- joint R_ankle_2: limit lower=-0.4886 upper=0.4886 effort=70 velocity=4.9 -> lower=-0.4014 upper=0.4014 effort=70 velocity=4.9
- joint R_hip_1: limit lower=-3.14 upper=3.14 effort=150 velocity=2.3 -> lower=-0.65 upper=0.83 effort=150 velocity=2.3
- joint R_hip_3: limit lower=-1.57 upper=1.57 effort=179 velocity=3.0 -> lower=-0.6 upper=1.57 effort=179 velocity=3.0
- joint R_shoulder_1: limit lower=-1.047 upper=2.44346 effort=150 velocity=3.14 -> lower=-1.04607 upper=2.44346 effort=150 velocity=3.14
- joint R_shoulder_2: limit lower=-0.7854 upper=1.082 effort=200 velocity=1.57 -> lower=-0.7854 upper=1.0472 effort=200 velocity=1.57
- joint R_wrist_1: limit lower=-0.663 upper=0.663 effort=30 velocity=3.42 -> lower=-0.63 upper=0.63 effort=30 velocity=3.42
- joint R_wrist_2: limit lower=-0.75 upper=0.75 effort=30 velocity=3.42 -> lower=-0.73 upper=0.73 effort=30 velocity=3.42
- joint waist_0: limit lower=-0.7 upper=0.1 effort=300 velocity=2.8 -> lower=-0.26 upper=0.26 effort=300 velocity=2.8

Commit message: updating the joint limits to those of the real robots (except for waist_0: the real robot will increase the range to 45 degrees from 18 degrees, shortly); verified the new limits to be ingress-compatible in bit-in-and-out controller commit 569c

File: urdf/bit_xuanyuan.urdf (robot description, URDF)
Before this commit: robot bit_xuanyuan, 44 links, 43 joints
Joints:
- joint L_ankle_1: limit lower=-0.4014 upper=0.4014 effort=116 velocity=4.3 -> lower=-0.436 upper=0.436 effort=116 velocity=4.3
- joint L_ankle_2: limit lower=-0.4014 upper=0.4014 effort=70 velocity=4.9 -> lower=-0.35 upper=0.35 effort=70 velocity=4.9
- joint L_hip_1: limit lower=-3.14 upper=3.14 effort=150 velocity=2.3 -> lower=-0.82 upper=0.64 effort=150 velocity=2.3
- joint L_knee_1: limit lower=-2.7925 upper=0.1919 effort=300 velocity=2.0 -> lower=-2.1 upper=0.01 effort=300 velocity=2.0
- joint L_knee_2: limit lower=-1.57 upper=1.57 effort=65 velocity=7.0 -> lower=-0.71 upper=0.71 effort=65 velocity=7.0
- joint R_ankle_1: limit lower=-0.4014 upper=0.4014 effort=116 velocity=4.3 -> lower=-0.436 upper=0.436 effort=116 velocity=4.3
- joint R_ankle_2: limit lower=-0.4014 upper=0.4014 effort=70 velocity=4.9 -> lower=-0.35 upper=0.35 effort=70 velocity=4.9
- joint R_hip_1: limit lower=-0.65 upper=0.83 effort=150 velocity=2.3 -> lower=-0.64 upper=0.82 effort=150 velocity=2.3
- joint R_knee_1: limit lower=-2.7925 upper=0.1919 effort=300 velocity=2.0 -> lower=-2.1 upper=0.01 effort=300 velocity=2.0
- joint R_knee_2: limit lower=-1.57 upper=1.57 effort=60 velocity=7.1 -> lower=-0.71 upper=0.71 effort=60 velocity=7.1
- joint waist_0: limit lower=-0.26 upper=0.26 effort=300 velocity=2.8 -> lower=-0.7 upper=0.26 effort=300 velocity=2.8

Commit message: corrected directions on L_shoulder_1

File: urdf/bit_xuanyuan.urdf (robot description, URDF)
Before this commit: robot bit_xuanyuan, 44 links, 43 joints
Joints:
- joint L_shoulder_1: axis 0 0 1 -> 0 0 -1; limit lower=-2.62 upper=0.7 effort=150 velocity=3.14 -> lower=-0.7 upper=2.62 effort=150 velocity=3.14

Commit message: temporarilly limited waist pitch forward angle limit for safety concern; remember to increase it before Ingress task

File: urdf/bit_xuanyuan.urdf (robot description, URDF)
Before this commit: robot bit_xuanyuan, 44 links, 43 joints
Joints:
- joint waist_0: limit lower=-0.4 upper=0.08 effort=300 velocity=2.8 -> lower=-0.35 upper=0.08 effort=300 velocity=2.8

Commit message: Update waist pitch limits

File: urdf/bit_xuanyuan.urdf (robot description, URDF)
Before this commit: robot bit_xuanyuan, 44 links, 43 joints
Joints:
- joint waist_0: limit lower=-0.7 upper=0.26 effort=300 velocity=2.8 -> lower=-0.4 upper=0.08 effort=300 velocity=2.8

Commit message: Update ankle limits

File: urdf/bit_xuanyuan.urdf (robot description, URDF)
Before this commit: robot bit_xuanyuan, 44 links, 43 joints
Joints:
- joint L_ankle_1: limit lower=-0.436 upper=0.436 effort=116 velocity=4.3 -> lower=-0.6 upper=0.436 effort=116 velocity=4.3
- joint R_ankle_1: limit lower=-0.436 upper=0.436 effort=116 velocity=4.3 -> lower=-0.436 upper=0.6 effort=116 velocity=4.3

Commit message: Change the root body to waist_1

File: urdf/bit_xuanyuan.urdf (robot description, URDF)
Before this commit: robot bit_xuanyuan, 44 links, 43 joints
Links:
- added link torso_tf
Joints:
- added joint torso_tf: type fixed, parent torso_tf, child torso, origin xyz=0 0.075 -0.075 rpy=-1.5707963267949 3.14 0
- joint L_hip_1: origin xyz=0 -0.0874524045087781 0.0804896286305103 rpy=0 0 1.5707963267949 -> xyz=0 0.0874524045087781 -0.08049 rpy=-3.14159265358979 0 -1.5707963267949
- joint R_hip_1: origin xyz=5.9130214832445E-05 0.0873497468913164 0.0804842516395254 rpy=0 0 1.5707963267949 -> xyz=0 -0.0874524045087781 -0.08049 rpy=-3.14159265358979 0 -1.5707963267949
- joint waist: child torso -> waist_1
- joint waist_0: axis 0 0 1 -> 0 0 -1; child waist_0 -> torso_tf; origin xyz=0 0.0751588565074892 -0.0749999999999999 rpy=1.5707963267949 0 3.14159265 -> xyz=0 0.0751588565074892 0.046 rpy=1.5707963267949 0 -3.14159265; parent torso -> waist_0
- joint waist_1: child waist_1 -> waist_0; origin xyz=0 -0.0460046428794829 -0.0751888646756264 rpy=1.5707963267949 3.1415926535 0 -> xyz=0 0 0 rpy=0 0 0; parent waist_0 -> waist_1

Commit message: Update joint limits

File: urdf/bit_xuanyuan.urdf (robot description, URDF)
Before this commit: robot bit_xuanyuan, 45 links, 44 joints
Joints:
- joint L_elbow_2: limit lower=-1.5075 upper=4.7728 effort=20 velocity=10.14 -> lower=-1.5075 upper=1.4835 effort=20 velocity=10.14

Commit message: decreased friction at both feet, and made gripper contact a bit softer

File: urdf/bit_xuanyuan.urdf (robot description, URDF)
Before this commit: robot bit_xuanyuan, 45 links, 44 joints
Joints:
- joint R_ankle_1: limit lower=-0.436 upper=0.6 effort=116 velocity=4.3 -> lower=-1.0 upper=1.0 effort=116 velocity=4.3

Commit message: updated joint limits in urdf according to the limit written in the robot's drivers; may need to loosen both limits later; also added self collision check btw right foot and left leg in the robot's minimal collision check set

File: urdf/bit_xuanyuan.urdf (robot description, URDF)
Before this commit: robot bit_xuanyuan, 45 links, 44 joints
Joints:
- joint L_elbow_1: limit lower=0 upper=1.745 effort=200 velocity=2.14 -> lower=-0.1 upper=1.745 effort=200 velocity=2.14
- joint L_gripper_1: limit lower=-0.01 upper=0.01 effort=200 velocity=0.03 -> lower=-0.042 upper=0.012 effort=200 velocity=0.03
- joint L_gripper_2: limit lower=-0.01 upper=0.01 effort=200 velocity=1 -> lower=-0.012 upper=0.042 effort=200 velocity=1
- joint L_shoulder_1: limit lower=-0.7 upper=2.62 effort=150 velocity=3.14 -> lower=-1.04 upper=2.44 effort=150 velocity=3.14
- joint R_elbow_1: limit lower=0 upper=1.745 effort=200 velocity=2.14 -> lower=-0.1 upper=1.745 effort=200 velocity=2.14
- joint R_gripper_1: limit lower=-0.01 upper=0.01 effort=200 velocity=0.03 -> lower=-0.0135 upper=0.009 effort=200 velocity=0.03
- joint R_gripper_2: limit lower=-0.01 upper=0.01 effort=200 velocity=1 -> lower=-0.009 upper=0.0135 effort=200 velocity=1

Commit message: increased joint range of waist_0 in one direction in the urdf

File: urdf/bit_xuanyuan.urdf (robot description, URDF)
Before this commit: robot bit_xuanyuan, 45 links, 44 joints
Joints:
- joint waist_0: limit lower=-0.35 upper=0.08 effort=300 velocity=2.8 -> lower=-0.68 upper=0.06 effort=300 velocity=2.8

Commit message: tentative changes to the ActualRobot; increased a few joint range; ignore gripper joint range as the coeffcient in reality and mujoco sim is different

File: urdf/bit_xuanyuan.urdf (robot description, URDF)
Before this commit: robot bit_xuanyuan, 45 links, 44 joints
Joints:
- joint L_ankle_1: limit lower=-0.6 upper=0.436 effort=116 velocity=4.3 -> lower=-0.8 upper=0.436 effort=116 velocity=4.3
- joint L_gripper_1: limit lower=-0.042 upper=0.012 effort=200 velocity=0.03 -> lower=-0.042 upper=0.05 effort=200 velocity=0.03
- joint L_gripper_2: limit lower=-0.012 upper=0.042 effort=200 velocity=1 -> lower=-0.05 upper=0.042 effort=200 velocity=1
- joint waist_0: limit lower=-0.68 upper=0.06 effort=300 velocity=2.8 -> lower=-0.88 upper=0.16 effort=300 velocity=2.8
- joint waist_1: limit lower=-0.872 upper=0.872 effort=220 velocity=2.5 -> lower=-0.972 upper=0.972 effort=220 velocity=2.5
