Commit message: increased elbow_1 range to fascilibat AdjustCoM after LandRightHip on the car seat

File: urdf/bit_xuanyuan.urdf (robot description, URDF)
Before this commit: robot bit_xuanyuan, 45 links, 44 joints
Joints:
- joint L_elbow_1: limit lower=-0.1 upper=1.745 effort=200 velocity=2.14 -> lower=-0.1 upper=2.245 effort=200 velocity=2.14
- joint R_elbow_1: limit lower=-0.1 upper=1.745 effort=200 velocity=2.14 -> lower=-0.1 upper=2.545 effort=200 velocity=2.14

Commit message: increased gripper range and leg_foot collision safe distance

File: urdf/bit_xuanyuan.urdf (robot description, URDF)
Before this commit: robot bit_xuanyuan, 45 links, 44 joints
Joints:
- joint L_gripper_1: limit lower=-0.042 upper=0.012 effort=200 velocity=0.03 -> lower=-0.042 upper=0.032 effort=200 velocity=0.03
- joint L_gripper_2: limit lower=-0.012 upper=0.042 effort=200 velocity=1 -> lower=-0.032 upper=0.042 effort=200 velocity=1

Commit message: R_ankle_1 limits were wrong!

File: urdf/bit_xuanyuan.urdf (robot description, URDF)
Before this commit: robot bit_xuanyuan, 45 links, 44 joints
Joints:
- joint R_ankle_1: limit lower=-1.0 upper=1.0 effort=116 velocity=4.3 -> lower=-0.436 upper=0.6 effort=116 velocity=4.3

Commit message: tentatively increased L_wrist range in one direction changed gripper installation orientatin

File: urdf/bit_xuanyuan.urdf (robot description, URDF)
Before this commit: robot bit_xuanyuan, 45 links, 44 joints
Joints:
- joint L_hand: origin xyz=0 0 -0.0150000000000001 rpy=0 0 3.14159265358979 -> xyz=0 0 -0.0150000000000001 rpy=0 0 1.57
- joint L_wrist_2: limit lower=-0.73 upper=0.73 effort=50 velocity=3.14 -> lower=-1.5 upper=0.73 effort=50 velocity=3.14

Commit message: increased joint limits for L_wrist and added compountJoint constrains accordingly

File: urdf/bit_xuanyuan.urdf (robot description, URDF)
Before this commit: robot bit_xuanyuan, 45 links, 44 joints
Joints:
- joint L_wrist_1: limit lower=-0.63 upper=0.63 effort=30 velocity=3.14 -> lower=-0.9 upper=0.9 effort=30 velocity=3.14
- joint L_wrist_2: limit lower=-1.5 upper=0.73 effort=50 velocity=3.14 -> lower=-1.74 upper=1.34 effort=50 velocity=3.14

Commit message: manually adjusted FZ offset for both feet

File: urdf/bit_xuanyuan.urdf (robot description, URDF)
Before this commit: robot bit_xuanyuan, 45 links, 44 joints
Joints:
- joint L_hand: origin xyz=0 0 -0.0150000000000001 rpy=0 0 1.57 -> xyz=0 0 -0.0150000000000001 rpy=0 0 1.74533
- joint L_wrist_1: limit lower=-0.9 upper=0.9 effort=30 velocity=3.14 -> lower=-0.63 upper=0.63 effort=30 velocity=3.14
- joint L_wrist_2: limit lower=-1.74 upper=1.34 effort=50 velocity=3.14 -> lower=-1.5 upper=1.12 effort=50 velocity=3.14
